File: TripComputer/kicad/TripComputer.kicad_pcb (KiCad board)
At the start: 2 copper layers, 1 part, among them U1 ESP32-DevKitC

Commit message: PCB Symbols
Parts:
- added U3: ~, Peter:ILI9488, F.Cu at (182.9, 73.8)
- moved U1 6.73 mm to (106.7, 48.3)
Connections:
- U1 pad 14: GND -> +3.3V
- U1 pad 26: unconnected-(U1-ADC2_CH0/GPIO4-Pad26) -> Net-(U1-ADC2_CH0/GPIO4)
- U1 pad 32: GND -> +3.3V
- U1 pad 38: GND -> +3.3V
Routing:
- net GND: track 56.9 -> 0.00 mm

Commit message: Kicad updates
Parts:
- added C1: 100n, Resistor_THT:R_Box_L8.4mm_W2.5mm_P5.08mm, F.Cu at (58.4, 48.3)
- added C2: 100n, Resistor_THT:R_Box_L8.4mm_W2.5mm_P5.08mm, F.Cu at (58.4, 55.9)
- added J1: Diag, Connector_PinHeader_1.00mm:PinHeader_1x03_P1.00mm_Vertical, F.Cu at (66.0, 79.3)
- added R1: 510R, Resistor_THT:R_Box_L8.4mm_W2.5mm_P5.08mm, F.Cu at (58.4, 63.5)
- added U2: ~, Connector_PinHeader_1.00mm:PinHeader_1x04_P1.00mm_Vertical, F.Cu at (83.8, 99.1)
- added U4: ~, Peter:L9637D, F.Cu at (85.3, 62.4)
Connections:
- U1 pad 13: unconnected-(U1-MTDI/GPIO12/ADC2_CH5-Pad13) -> Net-(U1-MTDI/GPIO12/ADC2_CH5)
- U1 pad 14: +3.3V -> GND
- U1 pad 15: unconnected-(U1-MTCK/GPIO13/ADC2_CH4-Pad15) -> Net-(U1-MTCK/GPIO13/ADC2_CH4)
- U1 pad 24: unconnected-(U1-ADC2_CH2/GPIO2-Pad24) -> Net-(U1-ADC2_CH0/GPIO4)
- U1 pad 30: unconnected-(U1-GPIO18-Pad30) -> Net-(U1-GPIO18)
- U1 pad 31: unconnected-(U1-GPIO19-Pad31) -> Net-(U1-GPIO19)
- U1 pad 32: +3.3V -> GND
- U1 pad 37: unconnected-(U1-GPIO23-Pad37) -> Net-(U1-GPIO23)
- U1 pad 38: +3.3V -> GND
- U3 pad 1: +3.3V -> unconnected-(U3-VCC-Pad1)
- U3 pad 2: +3.3V -> unconnected-(U3-GND-Pad2)
- U3 pad 3: unconnected-(U3-CS-Pad3) -> GND
- U3 pad 5: unconnected-(U3-DC-Pad5) -> Net-(U1-ADC2_CH0/GPIO4)
- U3 pad 6: unconnected-(U3-SDI-Pad6) -> Net-(U1-GPIO23)
- U3 pad 7: unconnected-(U3-SCK-Pad7) -> Net-(U1-GPIO18)
- U3 pad 8: unconnected-(U3-LED-Pad8) -> +3.3V
- U3 pad 9: unconnected-(U3-SDO-Pad9) -> Net-(U1-GPIO19)
Routing:
- net GND: track 0.00 -> 137.0 mm
- net +3.3V: track 0.00 -> 58.0 mm
- net Net-(J1-Pin_2): track 0.00 -> 39.1 mm
- net Net-(U1-GPIO23): track 0.00 -> 28.0 mm
- net Net-(J1-Pin_3): track 0.00 -> 21.3 mm
